File: I2C-7313-cTc.sch (EAGLE design)
At the start: 38 parts, among them CON1 CONNECTOR-I2CLEFT, IC1 MAX7313AEG, SW1 CTC-6PDT, SW2 CTC-4P3T

Commit message: 2.1-panel
Parts:
- added AD3, AD4, AD5, I2C-CABLE1: (no value), con-lstb:MA04-2
- added C4, C5: 0.1uF, SPCoast:CAP0805
- added C6: 220uF, SPCoast:CAP-POLPTH-5MM
- added CODEBUTTON1: (no value), SPCoast:CONNECTOR-M021X02-LOCK
- added CON2: CONNECTOR-I2CLEFT, SPCoast:CONNECTOR-I2CLEFT
- added IC2: MAX7313AEG, maxim:MAX7313AEG
- added LED-SIG-E1, LED-SIG-W1, LED-SW-N1: Green, SPCoast:LEDLED3MM
- added LED-SIG-S1: Red, SPCoast:LEDLED3MM
- added LED-SW-R1: Red/Orange, SPCoast:LEDLED3MM
- added MCLED1: (no value), SPCoast:JUMPER-2PTH_LOCK
- added MCSWITCH1: (no value), SPCoast:CONNECTOR-M025MM-LOCK
- added MODBOARDLEDS1: (no value), SPCoast:CONNECTOR-M06LOCK_LONGPADS
- added R17, R20, R22, R23, R24, R25: 82R, SPCoast:R0805-RES
- added R18, R19, R21: 56R, SPCoast:R0805-RES
- added R26, R27, R28, R29, R30, R31, R32: 10k, SPCoast:R0805-RES
- added SW3: CTC-4P3T, SPCoast:CTC-4P3T
- added SW4: CTC-6PDT, SPCoast:CTC-6PDT
- added VR2: 3v3, SPCoast:VREG_LM1117SOT223
- BOARD1: value BOARD100X150X2-NOHOLES -> (none)
Connections:
- new net N$10: MCLED1.1, R22.2
- new net N$11: MODBOARDLEDS1.2, R23.2
- new net N$12: MODBOARDLEDS1.4, R24.2
- new net N$13: MODBOARDLEDS1.6, R25.2
- new net N$14: LED-SW-N1.C, R21.2
- new net N$15: LED-SW-R1.C, R20.2
- new net N$16: LED-SIG-E1.C, R19.2
- new net N$17: LED-SIG-W1.C, R18.2
- new net N$18: LED-SIG-S1.C, R17.2
- new net SCL1: AD3.8, AD4.8, AD5.8, CON2.SCL, I2C-CABLE1.1, I2C-CABLE1.2, IC2.SLC
- new net SDA1: AD3.6, AD4.6, AD5.6, CON2.SDA, I2C-CABLE1.3, I2C-CABLE1.4, IC2.SDA
- net +3V3: now also AD3.4, AD4.4, AD5.4, C5.1, IC2.V+, LED-SIG-E1.A, LED-SIG-S1.A, LED-SIG-W1.A, LED-SW-N1.A, LED-SW-R1.A, MCLED1.2, R23.1, R24.1, R25.1, R26.1, R27.1, R28.1, R29.1, R30.1, R31.1, R32.1, VR2.OUT, VR2.OUT@1
- net +5V: now also C4.1, C6.+, CON2.V+, I2C-CABLE1.5, I2C-CABLE1.6, VR2.IN
- net AD0: now also AD3.1, AD3.3, AD3.5, AD3.7, IC2.AD0
- net AD1: now also AD4.1, AD4.3, AD4.5, AD4.7, IC2.AD1
- net AD2: now also AD5.1, AD5.3, AD5.5, AD5.7, IC2.AD2
- net CODE: now also CODEBUTTON1.1, IC2.P12, R32.2
- net GND: now also AD3.2, AD4.2, AD5.2, C4.2, C5.2, C6.-, CODEBUTTON1.2, CON2.GND, I2C-CABLE1.7, I2C-CABLE1.8, IC2.GND, MCSWITCH1.2, SW3.A, SW4.A, VR2.ADJ
- net LED-MC: now also IC2.P8, R22.1
- net LED-SIG-E: now also IC2.P13, R19.1
- net LED-SIG-S: now also IC2.P14, R18.1
- net LED-SIG-W: now also IC2.P15, R17.1
- net LED-SW-N: now also IC2.P0, R20.1
- net LED-SW-R: now also IC2.P1, R21.1
- net MB1: now also IC2.P3, MODBOARDLEDS1.1
- net MB2: now also IC2.P4, MODBOARDLEDS1.3
- net MB3: now also IC2.P5, MODBOARDLEDS1.5
- net MC: now also IC2.P2, MCSWITCH1.1, R26.2
- net SIG-E: now also IC2.P11, R31.2, SW3.A1
- net SIG-S: now also IC2.P10, R30.2, SW3.A2
- net SIG-W: now also IC2.P9, R29.2, SW3.A3
- net SW-N: now also IC2.P7, R28.2, SW4.A1
- net SW-R: now also IC2.P6, R27.2, SW4.A2
